File: pcb/pcb.kicad_sch (KiCad schematic)
At the start: 61 parts, among them J1 SW, J2 HEATER, J3 FAN, J4 BME280, J5 DISPLAY, J6 NTC, J7 POWER, Q1 IRFR9024NTRPBF, Q2 2n3904S-RTK/PS_C18536, Q3 2n3904S-RTK/PS_C18536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

Commit message: Work with schematics and pcb. update *.ioc files at project.
Parts:
- removed C13: 100uf, Capacitor_THT:CP_Radial_D8.0mm_P5.00mm, symbol Device:C_Polarized
- added H1, H2, H3, H4: MountingHole, MountingHole:MountingHole_3.2mm_M3_DIN965_Pad, symbol Mechanical:MountingHole
Connections:
- net +3.3V: now also J4.4 (Pin_4); no longer J4.1 (Pin_1)
- net GND: now also J2.2 (Pin_2), J3.2 (Pin_2), J4.1 (Pin_1), J6.2 (Pin_2); no longer J2.1 (Pin_1), J3.1 (Pin_1), J4.4 (Pin_4), J6.1 (Pin_1)
- net NTC: now also J6.1 (Pin_1); no longer J6.2 (Pin_2)
- net PWM_BUZZER: now also U1.29 (PA8); no longer U1.16 (PA6)
- net PWM_FAN: now also U1.40 (PB4); no longer U1.38 (PA15)
- net PWM_HEATER: now also U1.39 (PB3); no longer U1.29 (PA8)
- net at D1.1 (K), Q1.4 (D): now also J2.1 (Pin_1); no longer J2.2 (Pin_2)
- net at C14.1, D3.1 (K), U3.3 (D): now also J3.1 (Pin_1); no longer J3.2 (Pin_2)
Other:
- moved on the sheet: J2, J3, J6

Commit message: Update display ss1306 footprint. paste text refrenece on pcb
Connections:
- net +24V: now also J7.1 (Pin_1); no longer J7.2 (Pin_2)
- net GND: now also J2.1 (Pin_1), J6.1 (Pin_1), J7.2 (Pin_2); no longer J2.2 (Pin_2), J6.2 (Pin_2), J7.1 (Pin_1)
- net NTC: now also J6.2 (Pin_2); no longer J6.1 (Pin_1)
- net at D1.1 (K), Q1.4 (D): now also J2.2 (Pin_2); no longer J2.1 (Pin_1)
Other:
- moved on the sheet: J2, J6, J7
Changed lines of the file:
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@@
     )
   )
-  (symbol (lib_id "Connector:Conn_01x02_Pin") (at 279.4 241.3 0) (mirror y) (unit 1)
+  (symbol (lib_id "Connector:Conn_01x02_Pin") (at 279.4 243.84 180) (unit 1)
     (in_bom yes) (on_board yes) (dnp no)
-    (property "Reference" "J6" (at 280.67 243.84 0)
-      (effects (font (size 1.27 1.27)) (justify right))
-    )
-    (property "Value" "NTC" (at 280.67 241.3 0)
-      (effects (font (size 1.27 1.27)) (justify right))
-    )
-    (property "Footprint" "easyeda2kicad:CONN-TH_2P-P2.50_HC-XH-2A-G" (at 279.4 241.3 0)
-      (effects (font (size 1.27 1.27)) hide)
-    )
-    (property "Datasheet" "~" (at 279.4 241.3 0)
+    (property "Reference" "J6" (at 280.67 241.3 0)
+      (effects (font (size 1.27 1.27)) (justify right))
+    )
+    (property "Value" "NTC" (at 280.67 243.84 0)
+      (effects (font (size 1.27 1.27)) (justify right))
+    )
+    (property "Footprint" "easyeda2kicad:CONN-TH_2P-P2.50_HC-XH-2A-G" (at 279.4 243.84 0)
+      (effects (font (size 1.27 1.27)) hide)
+    )
+    (property "Datasheet" "~" (at 279.4 243.84 0)
       (effects (font (size 1.27 1.27)) hide)
     )
@@
     (in_bom yes) (on_board yes) (dnp no) (fields_autoplaced)
     (property "Reference" "H4" (at 73.66 220.98 0)
-      (effects (font (size 1.27 1.27)) (justify left))
+      (effects (font (size 1.27 1.27)) (justify left) hide)
     )
     (property "Value" "MountingHole" (at 73.66 223.52 0)
@@
     (in_bom yes) (on_board yes) (dnp no) (fields_autoplaced)
     (property "Reference" "H2" (at 73.66 208.28 0)
-      (effects (font (size 1.27 1.27)) (justify left))
+      (effects (font (size 1.27 1.27)) (justify left) hide)
     )
     (property "Value" "MountingHole" (at 73.66 210.82 0)
@@
     (in_bom yes) (on_board yes) (dnp no) (fields_autoplaced)
     (property "Reference" "H1" (at 73.66 201.93 0)
-      (effects (font (size 1.27 1.27)) (justify left))
+      (effects (font (size 1.27 1.27)) (justify left) hide)
     )
     (property "Value" "MountingHole" (at 73.66 204.47 0)
@@
     )
   )
-  (symbol (lib_id "Connector:Conn_01x02_Pin") (at 370.84 176.53 180) (unit 1)
+  (symbol (lib_id "Connector:Conn_01x02_Pin") (at 370.84 173.99 0) (mirror y) (unit 1)
     (in_bom yes) (on_board yes) (dnp no)
-    (property "Reference" "J7" (at 372.11 173.99 0)
-      (effects (font (size 1.27 1.27)) (justify right))
-    )
-    (property "Value" "POWER" (at 372.11 176.53 0)
-      (effects (font (size 1.27 1.27)) (justify right))
-    )
-    (property "Footprint" "TerminalBlock_Phoenix:TerminalBlock_Phoenix_MKDS-1,5-2_1x02_P5.00mm_Horizontal" (at 370.84 176.53 0)
-      (effects (font (size 1.27 1.27)) hide)
-    )
-    (property "Datasheet" "~" (at 370.84 176.53 0)
+    (property "Reference" "J7" (at 372.11 176.53 0)
+      (effects (font (size 1.27 1.27)) (justify right))
+    )
+    (property "Value" "POWER" (at 372.11 173.99 0)
+      (effects (font (size 1.27 1.27)) (justify right))
+    )
+    (property "Footprint" "TerminalBlock_Phoenix:TerminalBlock_Phoenix_MKDS-1,5-2_1x02_P5.00mm_Horizontal" (at 370.84 173.99 0)
+      (effects (font (size 1.27 1.27)) hide)
+    )
+    (property "Datasheet" "~" (at 370.84 173.99 0)
       (effects (font (size 1.27 1.27)) hide)
     )
@@
     )
   )
-  (symbol (lib_id "Connector:Conn_01x02_Pin") (at 367.03 67.31 0) (mirror y) (unit 1)
+  (symbol (lib_id "Connector:Conn_01x02_Pin") (at 367.03 69.85 180) (unit 1)
     (in_bom yes) (on_board yes) (dnp no)
-    (property "Reference" "J2" (at 368.3 69.85 0)
-      (effects (font (size 1.27 1.27)) (justify right))
-    )
-    (property "Value" "HEATER" (at 368.3 67.31 0)
-      (effects (font (size 1.27 1.27)) (justify right))
-    )
-    (property "Footprint" "TerminalBlock_Phoenix:TerminalBlock_Phoenix_MKDS-1,5-2_1x02_P5.00mm_Horizontal" (at 367.03 67.31 0)
-      (effects (font (size 1.27 1.27)) hide)
-    )
-    (property "Datasheet" "~" (at 367.03 67.31 0)
+    (property "Reference" "J2" (at 368.3 67.31 0)
+      (effects (font (size 1.27 1.27)) (justify right))
+    )
+    (property "Value" "HEATER" (at 368.3 69.85 0)
+      (effects (font (size 1.27 1.27)) (justify right))
+    )
+    (property "Footprint" "TerminalBlock_Phoenix:TerminalBlock_Phoenix_MKDS-1,5-2_1x02_P5.00mm_Horizontal" (at 367.03 69.85 0)
+      (effects (font (size 1.27 1.27)) hide)
+    )
+    (property "Datasheet" "~" (at 367.03 69.85 0)
       (effects (font (size 1.27 1.27)) hide)
     )
@@
     (in_bom yes) (on_board yes) (dnp no) (fields_autoplaced)
     (property "Reference" "H3" (at 73.66 214.63 0)
-      (effects (font (size 1.27 1.27)) (justify left))
+      (effects (font (size 1.27 1.27)) (justify left) hide)
     )
     (property "Value" "MountingHole" (at 73.66 217.17 0)
